File: board/TinyFPGA-A-Programmer.sch (KiCad schematic (older format))
At the start: 13 parts, among them J1 USB, J2 JTAG, J3 ICSP, J4 CONN_01X06, U1 PIC16F1455-QFN16, U2 MIC5504-3.3YM5-TR

Commit message: Change PIC footprint and shape
Parts:
- removed C4: 1uF, Capacitors_SMD:C_0603, symbol C
- removed U1: PIC16F1455-QFN16, Housings_DFN_QFN:QFN-16-1EP_4x4mm_Pitch0.65mm, symbol PIC16F1455-QFN16
- removed U2: MIC5504-3.3YM5-TR, TinyFPGA:SOT23, symbol MIC5504-3.3YM5-TR
- added C4: 1uF, Capacitor_SMD:C_0805_2012Metric_Pad1.15x1.40mm_HandSolder, symbol Device:C
- added U1: AP1117-33, Package_TO_SOT_SMD:SOT-223-3_TabPin2, symbol Regulator_Linear:AP1117-33
- added U2: PIC16F1455-ISL, Package_SO:SOIC-14_3.9x8.7mm_P1.27mm, symbol MCU_Microchip_PIC16:PIC16F1455-ISL
- C1, C2, C3: footprint Capacitors_SMD:C_0603 -> Capacitor_SMD:C_0805_2012Metric_Pad1.15x1.40mm_HandSolder; symbol C -> Device:C
- J1: footprint TinyFPGA:FCI-Micro-USB -> Connectors:629105150521; symbol USB_OTG -> TinyFPGA-A-Programmer-rescue:USB_OTG
- J2: footprint Pin_Headers:Pin_Header_Straight_1x05_Pitch2.54mm -> Connector_PinHeader_2.54mm:PinHeader_1x05_P2.54mm_Vertical; symbol CONN_01X05 -> TinyFPGA-A-Programmer-rescue:CONN_01X05
- J3, J4: footprint Pin_Headers:Pin_Header_Straight_1x06_Pitch2.54mm -> Connector_PinHeader_2.54mm:PinHeader_1x06_P2.54mm_Vertical; symbol CONN_01X06 -> TinyFPGA-A-Programmer-rescue:CONN_01X06
- TP1, TP2, TP3: footprint Measurement_Points:Measurement_Point_Round-SMD-Pad_Big -> TestPoint:TestPoint_Pad_D1.5mm; symbol TEST -> TinyFPGA-A-Programmer-rescue:TEST
Connections:
- net labels added: D+, D-, RC2, RC3, RC4, RC5
- wire segments 60 -> 61
Other:
- moved on the sheet: J1, J2, J3, J4, TP1, TP2, TP3
